Commit message: some work on rviz visualization

File: PraRobSem6/urdf/prarob_manipulator.xacro (robot description, xacro)
@@ -30,5 +30,5 @@
       <origin rpy="0 0 0" xyz="0 0 0"/>
       <geometry>
-        <mesh filename="package://ros2_prarob/meshes/postolje_seminar_v1.stl" scale="0.01 0.01 0.01"/>
+        <mesh filename="package://PraRobSem6/meshes/postolje_seminar_v1.stl" scale="0.01 0.01 0.01"/>
       </geometry>
       <material name="">
@@ -47,5 +47,5 @@
     <parent link="link1"/>
     <child link="link2"/>
-    <origin xyz="0.0 0.0 1.0" rpy="0 0 0"/>
+    <origin xyz="0.0 10.0 1.0" rpy="0 1.52 0"/>
     <axis xyz="0 0 1"/>
     <limit velocity="10.0" effort="1" lower="-2.82743338823" upper="2.82743338823" />
@@ -56,5 +56,5 @@
       <origin xyz="0 0 0.3" rpy="0 0 0"/>
       <geometry>
-        <box size="0.05 0.05 0.6"/>
+        <box size="0.7 0.5 0.84"/>
       </geometry>
       <color rgba="0 0.8 0.0 1"/>
@@ -63,5 +63,5 @@
       <origin xyz="0 0 0.3" rpy="0 0 0"/>
       <geometry>
-        <box size="0.05 0.05 0.6"/>
+        <box size="0.7 0.5 0.84"/>
       </geometry>
     </collision>
@@ -80,5 +80,5 @@
       <origin xyz="0.15 0 0" rpy="0 0 0"/>
       <geometry>
-        <box size="0.3 0.05 0.05"/>
+        <box size="2.0 0.12 0.3"/>
       </geometry>
       <color rgba="0 0 0.8 1"/>
@@ -91,5 +91,5 @@
     </collision>
   </link>
-  <!-- Joint 2 -->
+  <!-- Joint 3 -->
   <joint name="joint3" type="revolute">
     <parent link="link3"/>

Commit message: urdf + inverse kinematics + camera calibration

File: PraRobSem6/urdf/prarob_manipulator.xacro (robot description, xacro)
@@ -9,20 +9,4 @@
     <axis xyz="0 0 1" />
   </joint>
-  <!-- Link 1 - primitives-->
-  <!--link name="link1">
-    <visual>
-      <origin xyz="0 0 0.5" rpy="0 0 0"/>
-      <geometry>
-        <box size="0.05 0.05 1.0"/>
-      </geometry>
-      <color rgba="0 0 0.8 1"/>
-    </visual>
-    <collision>
-      <origin xyz="0 0 0" rpy="0 0 0"/>
-      <geometry>
-        <box size="0.05 0.05 1.0"/>
-      </geometry>
-    </collision>
-  </link-->
 <!-- Link 1 - stl -->
   <link name="link1">
@@ -30,14 +14,11 @@
       <origin rpy="0 0 0" xyz="0 0 0"/>
       <geometry>
-        <mesh filename="package://PraRobSem6/meshes/postolje_seminar_v1.stl" scale="0.01 0.01 0.01"/>
+        <mesh filename="package://PraRobSem6/meshes/postolje_i_baza.stl" scale="0.01 0.01 0.01"/>
       </geometry>
-      <material name="">
-        <color rgba="0.054901960784313725 0.054901960784313725 0.06274509803921569 1.0"/>
-      </material>
     </visual>
     <collision>
       <origin rpy="0 0 0" xyz="0 0 0"/>
       <geometry>
-        <mesh filename="package://ros2_prarob/meshes/postolje_seminar_v1.stl" scale="0.01 0.01 0.01"/>
+        <mesh filename="package://PraRobSem6/meshes/postolje_i_baza.stl" scale="0.01 0.01 0.01"/>
       </geometry>
     </collision>
@@ -47,5 +28,5 @@
     <parent link="link1"/>
     <child link="link2"/>
-    <origin xyz="0.0 10.0 1.0" rpy="0 1.52 0"/>
+    <origin xyz="0.0 0 0" rpy="0 0 0"/>
     <axis xyz="0 0 1"/>
     <limit velocity="10.0" effort="1" lower="-2.82743338823" upper="2.82743338823" />
@@ -54,14 +35,14 @@
   <link name="link2">
     <visual>
-      <origin xyz="0 0 0.3" rpy="0 0 0"/>
+      <origin xyz="0 0 0" rpy="0 0 0"/>
       <geometry>
-        <box size="0.7 0.5 0.84"/>
+        <mesh filename="package://PraRobSem6/meshes/prvi_zglob.stl" scale="0.01 0.01 0.01"/>
       </geometry>
       <color rgba="0 0.8 0.0 1"/>
     </visual>
     <collision>
-      <origin xyz="0 0 0.3" rpy="0 0 0"/>
+      <origin xyz="0 0 0" rpy="0 0 0"/>
       <geometry>
-        <box size="0.7 0.5 0.84"/>
+        <mesh filename="package://PraRobSem6/meshes/prvi_zglob.stl" scale="0.01 0.01 0.01"/>
       </geometry>
     </collision>
@@ -71,5 +52,5 @@
     <parent link="link2"/>
     <child link="link3"/>
-    <origin xyz="0.0 0.0 0.60" rpy="0 0 0"/>
+    <origin xyz="0.0 0.0 0" rpy="0 0 0"/>
     <axis xyz="1 0 0"/>
     <limit velocity="10.0" effort="1" lower="-2.82743338823" upper="2.82743338823" />
@@ -78,14 +59,14 @@
   <link name="link3">
     <visual>
-      <origin xyz="0.15 0 0" rpy="0 0 0"/>
+      <origin xyz="0 0 0" rpy="0 0 0"/>
       <geometry>
-        <box size="2.0 0.12 0.3"/>
+        <mesh filename="package://PraRobSem6/meshes/drugi_zglob.stl" scale="0.01 0.01 0.01"/>
       </geometry>
-      <color rgba="0 0 0.8 1"/>
+      <color rgba="0 0 0"/>
     </visual>
     <collision>
       <origin xyz="0 0 0" rpy="0 0 0"/>
       <geometry>
-        <box size="0.3 0.05 0.05"/>
+        <mesh filename="package://PraRobSem6/meshes/drugi_zglob.stl" scale="0.01 0.01 0.01"/>
       </geometry>
     </collision>
@@ -95,5 +76,5 @@
     <parent link="link3"/>
     <child link="link_tool"/>
-    <origin xyz="0.3 0.0 0.0" rpy="0 0 0"/>
+    <origin xyz="0 0 0" rpy="0 0 0"/>
     <axis xyz="1 0 0"/>
     <limit velocity="10.0" effort="1" lower="-2.82743338823" upper="2.82743338823" />
@@ -104,12 +85,12 @@
       <origin xyz="0 0 0" rpy="0 0 0"/>
       <geometry>
-        <box size="0.08 0.08 0.08"/>
+        <mesh filename="package://PraRobSem6/meshes/treci_zglob.stl" scale="0.01 0.01 0.01"/>
       </geometry>
-      <color rgba="0 0 0.8 1"/>
+      <color rgba="255 104 255 1"/>
     </visual>
     <collision>
       <origin xyz="0 0 0" rpy="0 0 0"/>
       <geometry>
-        <box size="0.08 0.08 0.08"/>
+        <mesh filename="package://PraRobSem6/meshes/treci_zglob.stl" scale="0.01 0.01 0.01"/>
       </geometry>
     </collision>

Commit message: urdf

File: PraRobSem6/urdf/prarob_manipulator.xacro (robot description, xacro)
@@ -12,5 +12,5 @@
   <link name="link1">
     <visual>
-      <origin rpy="0 0 0" xyz="0 0 0"/>
+      <origin rpy="0 0 0" xyz="0 0 0.0435"/>
       <geometry>
         <mesh filename="package://PraRobSem6/meshes/postolje_i_baza.stl" scale="0.01 0.01 0.01"/>
@@ -28,5 +28,5 @@
     <parent link="link1"/>
     <child link="link2"/>
-    <origin xyz="0.0 0 0" rpy="0 0 0"/>
+    <origin xyz="0 0 0.087" rpy="0 0 0"/>
     <axis xyz="0 0 1"/>
     <limit velocity="10.0" effort="1" lower="-2.82743338823" upper="2.82743338823" />
@@ -35,12 +35,14 @@
   <link name="link2">
     <visual>
-      <origin xyz="0 0 0" rpy="0 0 0"/>
+      <origin xyz="0 0 0.005" rpy="0 0 0"/>
       <geometry>
         <mesh filename="package://PraRobSem6/meshes/prvi_zglob.stl" scale="0.01 0.01 0.01"/>
       </geometry>
-      <color rgba="0 0.8 0.0 1"/>
+      <material name="">
+        <color rgba="0 0 0 1.0"/>
+      </material>
     </visual>
     <collision>
-      <origin xyz="0 0 0" rpy="0 0 0"/>
+      <origin xyz="0 0 0.005" rpy="0 0 0"/>
       <geometry>
         <mesh filename="package://PraRobSem6/meshes/prvi_zglob.stl" scale="0.01 0.01 0.01"/>
@@ -52,6 +54,6 @@
     <parent link="link2"/>
     <child link="link3"/>
-    <origin xyz="0.0 0.0 0" rpy="0 0 0"/>
-    <axis xyz="1 0 0"/>
+    <origin xyz="0 0 0" rpy="0 0 0"/>
+    <axis xyz="0 1 0"/>
     <limit velocity="10.0" effort="1" lower="-2.82743338823" upper="2.82743338823" />
   </joint>
@@ -59,5 +61,5 @@
   <link name="link3">
     <visual>
-      <origin xyz="0 0 0" rpy="0 0 0"/>
+      <origin xyz="0 0 0.1" rpy="0 0 0"/>
       <geometry>
         <mesh filename="package://PraRobSem6/meshes/drugi_zglob.stl" scale="0.01 0.01 0.01"/>
@@ -66,5 +68,5 @@
     </visual>
     <collision>
-      <origin xyz="0 0 0" rpy="0 0 0"/>
+      <origin xyz="0 0 0.1" rpy="0 0 0"/>
       <geometry>
         <mesh filename="package://PraRobSem6/meshes/drugi_zglob.stl" scale="0.01 0.01 0.01"/>
@@ -76,6 +78,6 @@
     <parent link="link3"/>
     <child link="link_tool"/>
-    <origin xyz="0 0 0" rpy="0 0 0"/>
-    <axis xyz="1 0 0"/>
+    <origin xyz="0 0 0.2" rpy="0 0 0"/>
+    <axis xyz="0 1 0"/>
     <limit velocity="10.0" effort="1" lower="-2.82743338823" upper="2.82743338823" />
   </joint>
@@ -83,5 +85,5 @@
   <link name="link_tool">
     <visual>
-      <origin xyz="0 0 0" rpy="0 0 0"/>
+      <origin xyz="0 0 0.0825" rpy="0 0 0"/>
       <geometry>
         <mesh filename="package://PraRobSem6/meshes/treci_zglob.stl" scale="0.01 0.01 0.01"/>
@@ -90,5 +92,5 @@
     </visual>
     <collision>
-      <origin xyz="0 0 0" rpy="0 0 0"/>
+      <origin xyz="0 0 0.0825" rpy="0 0 0"/>
       <geometry>
         <mesh filename="package://PraRobSem6/meshes/treci_zglob.stl" scale="0.01 0.01 0.01"/>

Commit message: urdf 2

File: PraRobSem6/urdf/prarob_manipulator.xacro (robot description, xacro)
@@ -28,5 +28,5 @@
     <parent link="link1"/>
     <child link="link2"/>
-    <origin xyz="0 0 0.087" rpy="0 0 0"/>
+    <origin xyz="0 0.147 0.36" rpy="0 0 0"/>
     <axis xyz="0 0 1"/>
     <limit velocity="10.0" effort="1" lower="-2.82743338823" upper="2.82743338823" />
@@ -35,5 +35,5 @@
   <link name="link2">
     <visual>
-      <origin xyz="0 0 0.005" rpy="0 0 0"/>
+      <origin xyz="0 -0.147 -0.36" rpy="0 0 0"/>
       <geometry>
         <mesh filename="package://PraRobSem6/meshes/prvi_zglob.stl" scale="0.01 0.01 0.01"/>
@@ -44,5 +44,5 @@
     </visual>
     <collision>
-      <origin xyz="0 0 0.005" rpy="0 0 0"/>
+      <origin xyz="0 -0.147 -0.36" rpy="0 0 0"/>
       <geometry>
         <mesh filename="package://PraRobSem6/meshes/prvi_zglob.stl" scale="0.01 0.01 0.01"/>
@@ -54,6 +54,6 @@
     <parent link="link2"/>
     <child link="link3"/>
-    <origin xyz="0 0 0" rpy="0 0 0"/>
-    <axis xyz="0 1 0"/>
+    <origin xyz="0 0 0.55" rpy="0 0 0"/>
+    <axis xyz="0 0 1"/>
     <limit velocity="10.0" effort="1" lower="-2.82743338823" upper="2.82743338823" />
   </joint>
@@ -61,5 +61,5 @@
   <link name="link3">
     <visual>
-      <origin xyz="0 0 0.1" rpy="0 0 0"/>
+      <origin xyz="0 0 -0.55" rpy="0 0 0"/>
       <geometry>
         <mesh filename="package://PraRobSem6/meshes/drugi_zglob.stl" scale="0.01 0.01 0.01"/>
@@ -68,5 +68,5 @@
     </visual>
     <collision>
-      <origin xyz="0 0 0.1" rpy="0 0 0"/>
+      <origin xyz="0 0 -0.55" rpy="0 0 0"/>
       <geometry>
         <mesh filename="package://PraRobSem6/meshes/drugi_zglob.stl" scale="0.01 0.01 0.01"/>
@@ -78,6 +78,6 @@
     <parent link="link3"/>
     <child link="link_tool"/>
-    <origin xyz="0 0 0.2" rpy="0 0 0"/>
-    <axis xyz="0 1 0"/>
+    <origin xyz="0 1.78 0" rpy="0 0 0"/>
+    <axis xyz="0 0 1"/>
     <limit velocity="10.0" effort="1" lower="-2.82743338823" upper="2.82743338823" />
   </joint>
@@ -85,5 +85,5 @@
   <link name="link_tool">
     <visual>
-      <origin xyz="0 0 0.0825" rpy="0 0 0"/>
+      <origin xyz="0 -1.78 0" rpy="0 0 0"/>
       <geometry>
         <mesh filename="package://PraRobSem6/meshes/treci_zglob.stl" scale="0.01 0.01 0.01"/>
@@ -92,5 +92,5 @@
     </visual>
     <collision>
-      <origin xyz="0 0 0.0825" rpy="0 0 0"/>
+      <origin xyz="0 -1.78 0" rpy="0 0 0"/>
       <geometry>
         <mesh filename="package://PraRobSem6/meshes/treci_zglob.stl" scale="0.01 0.01 0.01"/>
